Commit message: added camera attached to camera mount

File: devastator_description/urdf/devastator_full.urdf.xacro (robot description, xacro)
@@ -1,6 +1,4 @@
 <?xml version="1.0"?>
 <robot name="devastator" xmlns:xacro="http://www.ros.org/wiki/xacro">
-  <xacro:property name="cameraSize" value="0.025"/>
-  <xacro:property name="cameraMass" value="0.1"/>
   <xacro:include filename="$(find devastator)/devastator_description/urdf/devastator_laser.gazebo.xacro" />
   <!--xacro:include filename="$(find mybot_description)/urdf/materials.xacro" /-->
@@ -348,12 +346,12 @@
 	<child link="camera_pan"/>
 	<origin xyz="0.0545 0  0.1125" rpy="0 0 0"/>
-    <limit effort="1000.0" lower="0.0" upper="3.1416" velocity="0.5"/>
+    <limit effort="1000.0" lower="0.0" upper="6.2831" velocity="0.5"/>
 	<axis xyz="0 0 1"/>
 </joint>
-<!--link name="camera">
+<link name="camera">
     <collision>
       <origin xyz="0 0 0" rpy="0 0 0"/>
       <geometry>
-        <box size="${cameraSize} ${cameraSize} ${cameraSize}"/>
+        <box size="0.005 0.01 0.01"/>
       </geometry>
     </collision>
@@ -361,11 +359,11 @@
       <origin xyz="0 0 0" rpy="0 0 0"/>
       <geometry>
-        <mesh filename="package://devastator/devastator_description/meshes/sensors/hokuyo.dae"/>
+        <mesh filename="package://devastator/devastator_description/meshes/sensors/camera.dae"/>
       </geometry>
 	</visual>
     <inertial>
-      <mass value="${cameraMass}" />
-      <origin xyz="0 0 0" rpy="0 0 0"/>
-      <box_inertia m="${cameraMass}" x="${cameraSize}" y="${cameraSize}" z="${cameraSize}" />
+      <mass value="0.25" />
+      <origin xyz="0 0 0" rpy="0 0 0"/>
+      <box_inertia m="0.25" x="0.015" y="0.015" z="0.02" />
       <inertia ixx="1.0e-6" ixy="0.0" ixz="0.0"
 	  iyy="1.0e-6" iyz="0.0" izz="1.0e-6" />
@@ -374,9 +372,9 @@
   <joint name="camera_joint" type="fixed">
     <axis xyz="0 1 0" />
-	<origin xyz="0.12 0 0.05" rpy="0 0 0"/>
-    <parent link="base_link"/>
+	<origin xyz="0.00625 0 0.01" rpy="0 0 0"/>
+    <parent link="camera_pan"/>
     <child link="camera"/>
   </joint>
-<link name="hokuyo">
+<!--link name="hokuyo">
     <collision>
       <origin xyz="0 0 0" rpy="0 0 0"/>

Commit message: Created new rviz file, added back digital IR sensors

File: devastator_description/urdf/devastator_full.urdf.xacro (robot description, xacro)
@@ -376,4 +376,58 @@
     <child link="camera"/>
   </joint>
+  <link name="dIR_BR">
+      <collision>
+        <origin xyz="0 0 0.0085" rpy="0 0 0"/>
+        <geometry>
+          <cylinder length="0.017" radius="0.0045"/>
+        </geometry>
+      </collision>
+      <visual>
+        <origin xyz="0 0 0" rpy="0 0 0"/>
+        <geometry>
+          <mesh filename="package://devastator/devastator_description/meshes/sensors/digital_ir.dae"/>
+        </geometry>
+  	</visual>
+      <inertial>
+        <mass value="0.25" />
+        <origin xyz="0 0 0" rpy="0 0 0"/>
+        <box_inertia m="0.25" x="0.015" y="0.015" z="0.02" />
+        <inertia ixx="1.0e-6" ixy="0.0" ixz="0.0"
+  	  iyy="1.0e-6" iyz="0.0" izz="1.0e-6" />
+      </inertial>
+  </link>
+    <joint name="dIR_BR_joint" type="fixed">
+      <axis xyz="0 1 0" />
+  	<origin xyz="-0.11676 0.05761 0.06139" rpy="0 -1.57 0"/>
+      <parent link="base_link"/>
+      <child link="dIR_BR"/>
+    </joint>
+    <link name="dIR_BL">
+        <collision>
+          <origin xyz="0 0 0.0085" rpy="0 0 0"/>
+          <geometry>
+            <cylinder length="0.017" radius="0.0045"/>
+          </geometry>
+        </collision>
+        <visual>
+          <origin xyz="0 0 0" rpy="0 0 0"/>
+          <geometry>
+            <mesh filename="package://devastator/devastator_description/meshes/sensors/digital_ir.dae"/>
+          </geometry>
+      </visual>
+        <inertial>
+          <mass value="0.25" />
+          <origin xyz="0 0 0" rpy="0 0 0"/>
+          <box_inertia m="0.25" x="0.015" y="0.015" z="0.02" />
+          <inertia ixx="1.0e-6" ixy="0.0" ixz="0.0"
+        iyy="1.0e-6" iyz="0.0" izz="1.0e-6" />
+        </inertial>
+    </link>
+      <joint name="dIR_BL_joint" type="fixed">
+        <axis xyz="0 1 0" />
+      <origin xyz="-0.11676 -0.05761 0.06139" rpy="0 -1.57 0"/>
+        <parent link="base_link"/>
+        <child link="dIR_BL"/>
+      </joint>
 <!--link name="hokuyo">
     <collision>

Commit message: Added analog front  IR sensors

File: devastator_description/urdf/devastator_full.urdf.xacro (robot description, xacro)
@@ -4,10 +4,5 @@
   <!--xacro:include filename="$(find mybot_description)/urdf/materials.xacro" /-->
   <xacro:include filename="$(find mybot_description)/urdf/macros.xacro" />
-<!--link name="base_footprint"/>
-  <joint name="base_joint" type="fixed">
-    <parent link="base_footprint"/>
-    <origin xyz="0.0 0.0 0.0" rpy="0 0 1.57"/>
-    <child link="base_link"/>
-  </joint-->
+<!--ROBOT BASE-->
 <link name="base_link">
 	<visual>
@@ -31,5 +26,5 @@
 	</inertial>
 </link>
-<!-- Right Wheels -->
+<!-- RIGHT WHEELS -->
 <link name="wheel_one_right">
 	<visual>
@@ -146,4 +141,5 @@
 	<axis xyz="0 1 0"/>
 </joint>
+<!--LEFT WHEELS-->
 <link name="wheel_one_left">
 	<visual>
@@ -320,9 +316,10 @@
 	<axis xyz="0 0 1"/>
 </joint>
+<!--SENSORS/ACCESSORIES-->
 <link name="camera_pan">
   <collision>
     <origin xyz="0 0 0" rpy="0 0 0"/>
     <geometry>
-      <!-- box size ="width lengtht height"-->
+    <!-- box size ="width lengtht height"-->
       <box size="0.01 0.025 0.03"/>
     </geometry>
@@ -333,101 +330,157 @@
       <mesh filename="package://devastator/devastator_description/meshes/base/camera_pan.dae"/>
     </geometry>
-</visual>
+  </visual>
   <!--inertial>
-    <mass value="${cameraMass}" />
-    <origin xyz="0 0 0" rpy="0 0 0"/>
-    <box_inertia m="${cameraMass}" x="${cameraSize}" y="${cameraSize}" z="${cameraSize}" />
+  <mass value="${cameraMass}" />
+  <origin xyz="0 0 0" rpy="0 0 0"/>
+  <box_inertia m="${cameraMass}" x="${cameraSize}" y="${cameraSize}" z="${cameraSize}" />
+  <inertia ixx="1.0e-6" ixy="0.0" ixz="0.0"
+  iyy="1.0e-6" iyz="0.0" izz="1.0e-6" />
+  </inertial-->
+</link>
+<joint name="camera_pan_joint" type="revolute">
+  <parent link="base_link"/>
+  <child link="camera_pan"/>
+  <origin xyz="0.0545 0  0.1125" rpy="0 0 0"/>
+  <limit effort="1000.0" lower="0.0" upper="6.2831" velocity="0.5"/>
+  <axis xyz="0 0 1"/>
+</joint>
+<link name="camera">
+  <collision>
+    <origin xyz="0 0 0" rpy="0 0 0"/>
+    <geometry>
+      <box size="0.005 0.01 0.01"/>
+    </geometry>
+  </collision>
+  <visual>
+    <origin xyz="0 0 0" rpy="0 0 0"/>
+    <geometry>
+      <mesh filename="package://devastator/devastator_description/meshes/sensors/camera.dae"/>
+    </geometry>
+  </visual>
+  <inertial>
+    <mass value="0.25" />
+    <origin xyz="0 0 0" rpy="0 0 0"/>
+    <box_inertia m="0.25" x="0.015" y="0.015" z="0.02" />
     <inertia ixx="1.0e-6" ixy="0.0" ixz="0.0"
-  iyy="1.0e-6" iyz="0.0" izz="1.0e-6" />
-</inertial-->
-</link>
-<joint name="camera_pan_joint" type="revolute">
-	<parent link="base_link"/>
-	<child link="camera_pan"/>
-	<origin xyz="0.0545 0  0.1125" rpy="0 0 0"/>
-    <limit effort="1000.0" lower="0.0" upper="6.2831" velocity="0.5"/>
-	<axis xyz="0 0 1"/>
-</joint>
-<link name="camera">
-    <collision>
-      <origin xyz="0 0 0" rpy="0 0 0"/>
-      <geometry>
-        <box size="0.005 0.01 0.01"/>
-      </geometry>
-    </collision>
-    <visual>
-      <origin xyz="0 0 0" rpy="0 0 0"/>
-      <geometry>
-        <mesh filename="package://devastator/devastator_description/meshes/sensors/camera.dae"/>
-      </geometry>
-	</visual>
-    <inertial>
-      <mass value="0.25" />
-      <origin xyz="0 0 0" rpy="0 0 0"/>
-      <box_inertia m="0.25" x="0.015" y="0.015" z="0.02" />
-      <inertia ixx="1.0e-6" ixy="0.0" ixz="0.0"
-	  iyy="1.0e-6" iyz="0.0" izz="1.0e-6" />
-    </inertial>
-</link>
-  <joint name="camera_joint" type="fixed">
-    <axis xyz="0 1 0" />
-	<origin xyz="0.00625 0 0.01" rpy="0 0 0"/>
-    <parent link="camera_pan"/>
-    <child link="camera"/>
-  </joint>
-  <link name="dIR_BR">
-      <collision>
-        <origin xyz="0 0 0.0085" rpy="0 0 0"/>
-        <geometry>
-          <cylinder length="0.017" radius="0.0045"/>
-        </geometry>
-      </collision>
-      <visual>
-        <origin xyz="0 0 0" rpy="0 0 0"/>
-        <geometry>
-          <mesh filename="package://devastator/devastator_description/meshes/sensors/digital_ir.dae"/>
-        </geometry>
-  	</visual>
-      <inertial>
-        <mass value="0.25" />
-        <origin xyz="0 0 0" rpy="0 0 0"/>
-        <box_inertia m="0.25" x="0.015" y="0.015" z="0.02" />
-        <inertia ixx="1.0e-6" ixy="0.0" ixz="0.0"
-  	  iyy="1.0e-6" iyz="0.0" izz="1.0e-6" />
-      </inertial>
-  </link>
-    <joint name="dIR_BR_joint" type="fixed">
-      <axis xyz="0 1 0" />
-  	<origin xyz="-0.11676 0.05761 0.06139" rpy="0 -1.57 0"/>
-      <parent link="base_link"/>
-      <child link="dIR_BR"/>
-    </joint>
-    <link name="dIR_BL">
-        <collision>
-          <origin xyz="0 0 0.0085" rpy="0 0 0"/>
-          <geometry>
-            <cylinder length="0.017" radius="0.0045"/>
-          </geometry>
-        </collision>
-        <visual>
-          <origin xyz="0 0 0" rpy="0 0 0"/>
-          <geometry>
-            <mesh filename="package://devastator/devastator_description/meshes/sensors/digital_ir.dae"/>
-          </geometry>
-      </visual>
-        <inertial>
-          <mass value="0.25" />
-          <origin xyz="0 0 0" rpy="0 0 0"/>
-          <box_inertia m="0.25" x="0.015" y="0.015" z="0.02" />
-          <inertia ixx="1.0e-6" ixy="0.0" ixz="0.0"
-        iyy="1.0e-6" iyz="0.0" izz="1.0e-6" />
-        </inertial>
-    </link>
-      <joint name="dIR_BL_joint" type="fixed">
-        <axis xyz="0 1 0" />
-      <origin xyz="-0.11676 -0.05761 0.06139" rpy="0 -1.57 0"/>
-        <parent link="base_link"/>
-        <child link="dIR_BL"/>
-      </joint>
+    iyy="1.0e-6" iyz="0.0" izz="1.0e-6" />
+  </inertial>
+</link>
+<joint name="camera_joint" type="fixed">
+  <axis xyz="0 1 0" />
+  <origin xyz="0.00625 0 0.01" rpy="0 0 0"/>
+  <parent link="camera_pan"/>
+  <child link="camera"/>
+</joint>
+<link name="dIR_BR">
+  <collision>
+  <origin xyz="0 0 0.0085" rpy="0 0 0"/>
+  <geometry>
+    <cylinder length="0.017" radius="0.0045"/>
+  </geometry>
+  </collision>
+  <visual>
+  <origin xyz="0 0 0" rpy="0 0 0"/>
+  <geometry>
+    <mesh filename="package://devastator/devastator_description/meshes/sensors/digital_ir.dae"/>
+  </geometry>
+  </visual>
+  <inertial>
+    <mass value="0.25" />
+    <origin xyz="0 0 0" rpy="0 0 0"/>
+    <box_inertia m="0.25" x="0.015" y="0.015" z="0.02" />
+    <inertia ixx="1.0e-6" ixy="0.0" ixz="0.0"
+    iyy="1.0e-6" iyz="0.0" izz="1.0e-6" />
+  </inertial>
+</link>
+<joint name="dIR_BR_joint" type="fixed">
+  <axis xyz="0 1 0" />
+  <origin xyz="-0.11676 0.05761 0.06139" rpy="0 -1.57 0"/>
+  <parent link="base_link"/>
+  <child link="dIR_BR"/>
+</joint>
+<link name="dIR_BL">
+  <collision>
+    <origin xyz="0 0 0.0085" rpy="0 0 0"/>
+    <geometry>
+      <cylinder length="0.017" radius="0.0045"/>
+    </geometry>
+  </collision>
+  <visual>
+    <origin xyz="0 0 0" rpy="0 0 0"/>
+    <geometry>
+      <mesh filename="package://devastator/devastator_description/meshes/sensors/digital_ir.dae"/>
+    </geometry>
+  </visual>
+  <inertial>
+    <mass value="0.25" />
+    <origin xyz="0 0 0" rpy="0 0 0"/>
+    <box_inertia m="0.25" x="0.015" y="0.015" z="0.02" />
+    <inertia ixx="1.0e-6" ixy="0.0" ixz="0.0"
+    iyy="1.0e-6" iyz="0.0" izz="1.0e-6" />
+  </inertial>
+</link>
+<joint name="dIR_BL_joint" type="fixed">
+  <axis xyz="0 1 0" />
+  <origin xyz="-0.11676 -0.05761 0.06139" rpy="0 -1.57 0"/>
+  <parent link="base_link"/>
+  <child link="dIR_BL"/>
+</joint>
+<link name="aIR_FR">
+  <collision>
+    <origin xyz="0 0 0" rpy="0 0 0"/>
+    <geometry>
+      <box size="0.01418 0.04839 0.013"/>
+    </geometry>
+  </collision>
+  <visual>
+    <origin xyz="0 0 0" rpy="0 0 0"/>
+    <geometry>
+      <mesh filename="package://devastator/devastator_description/meshes/sensors/analog_ir.dae"/>
+    </geometry>
+  </visual>
+  <inertial>
+    <mass value="0.25" />
+    <origin xyz="0 0 0" rpy="0 0 0"/>
+    <box_inertia m="0.25" x="0.015" y="0.015" z="0.02" />
+    <inertia ixx="1.0e-6" ixy="0.0" ixz="0.0"
+    iyy="1.0e-6" iyz="0.0" izz="1.0e-6" />
+  </inertial>
+</link>
+<joint name="aIR_FR_joint" type="revolute">
+  <axis xyz="0 0 1" />
+  <origin xyz="0.09648 -0.06266 0.06481" rpy="0 0 -0.7217"/>
+  <limit effort="1000.0" lower="0.0" upper="1.2217" velocity="0.5"/>
+  <parent link="base_link"/>
+  <child link="aIR_FR"/>
+</joint>
+<link name="aIR_FL">
+  <collision>
+    <origin xyz="0 0 0" rpy="0 0 0"/>
+    <geometry>
+      <box size="0.01418 0.04839 0.013"/>
+    </geometry>
+  </collision>
+  <visual>
+    <origin xyz="0 0 0" rpy="0 0 0"/>
+    <geometry>
+      <mesh filename="package://devastator/devastator_description/meshes/sensors/analog_ir.dae"/>
+    </geometry>
+  </visual>
+  <inertial>
+    <mass value="0.25" />
+    <origin xyz="0 0 0" rpy="0 0 0"/>
+    <box_inertia m="0.25" x="0.015" y="0.015" z="0.02" />
+    <inertia ixx="1.0e-6" ixy="0.0" ixz="0.0"
+    iyy="1.0e-6" iyz="0.0" izz="1.0e-6" />
+  </inertial>
+</link>
+<joint name="aIR_FL_joint" type="revolute">
+  <axis xyz="0 0 1" />
+  <origin xyz="0.09648 0.06266 0.06481" rpy="0 0 0.7217"/>
+  <limit effort="1000.0" lower="-1.2217" upper="0.0" velocity="0.5"/>
+  <parent link="base_link"/>
+  <child link="aIR_FL"/>
+</joint>
 <!--link name="hokuyo">
     <collision>

Commit message: changed digital IR model added ultrasonic and front dig IR sensor, adjust collision meshes

File: devastator_description/urdf/devastator_full.urdf.xacro (robot description, xacro)
@@ -373,9 +373,10 @@
   <child link="camera"/>
 </joint>
-<link name="dIR_BR">
-  <collision>
-  <origin xyz="0 0 0.0085" rpy="0 0 0"/>
+<link name="dIR_BL">
+  <collision>
+    <axis xyz="0 0 0" />
+    <origin xyz="0.0085 0 0" rpy="0 1.57 0"/>
   <geometry>
-    <cylinder length="0.017" radius="0.0045"/>
+    <cylinder  length="0.017" radius="0.0045" />
   </geometry>
   </collision>
@@ -394,40 +395,41 @@
   </inertial>
 </link>
+<joint name="dIR_BL_joint" type="fixed">
+  <axis xyz="0 1 0" />
+  <origin xyz="-0.11676 0.05761 0.06139" rpy="0 3.1416 0"/>
+  <parent link="base_link"/>
+  <child link="dIR_BL"/>
+</joint>
+<link name="dIR_BR">
+  <collision>
+    <axis xyz="0 1 0" />
+    <origin xyz="0.0085 0 0" rpy="0 1.57 0"/>
+    <geometry>
+      <cylinder radius="0.0045" length="0.017" />
+    </geometry>
+  </collision>
+  <visual>
+    <origin xyz="0 0 0" rpy="0 0 0"/>
+    <geometry>
+      <mesh filename="package://devastator/devastator_description/meshes/sensors/digital_ir.dae"/>
+    </geometry>
+  </visual>
+  <inertial>
+    <mass value="0.25" />
+    <origin xyz="0 0 0" rpy="0 0 0"/>
+    <box_inertia m="0.25" x="0.015" y="0.015" z="0.02" />
+    <inertia ixx="1.0e-6" ixy="0.0" ixz="0.0"
+    iyy="1.0e-6" iyz="0.0" izz="1.0e-6" />
+  </inertial>
+</link>
 <joint name="dIR_BR_joint" type="fixed">
   <axis xyz="0 1 0" />
-  <origin xyz="-0.11676 0.05761 0.06139" rpy="0 -1.57 0"/>
+  <origin xyz="-0.11676 -0.05761 0.06139" rpy="0 3.1416 0"/>
   <parent link="base_link"/>
   <child link="dIR_BR"/>
 </joint>
-<link name="dIR_BL">
-  <collision>
-    <origin xyz="0 0 0.0085" rpy="0 0 0"/>
-    <geometry>
-      <cylinder length="0.017" radius="0.0045"/>
-    </geometry>
-  </collision>
-  <visual>
-    <origin xyz="0 0 0" rpy="0 0 0"/>
-    <geometry>
-      <mesh filename="package://devastator/devastator_description/meshes/sensors/digital_ir.dae"/>
-    </geometry>
-  </visual>
-  <inertial>
-    <mass value="0.25" />
-    <origin xyz="0 0 0" rpy="0 0 0"/>
-    <box_inertia m="0.25" x="0.015" y="0.015" z="0.02" />
-    <inertia ixx="1.0e-6" ixy="0.0" ixz="0.0"
-    iyy="1.0e-6" iyz="0.0" izz="1.0e-6" />
-  </inertial>
-</link>
-<joint name="dIR_BL_joint" type="fixed">
-  <axis xyz="0 1 0" />
-  <origin xyz="-0.11676 -0.05761 0.06139" rpy="0 -1.57 0"/>
-  <parent link="base_link"/>
-  <child link="dIR_BL"/>
-</joint>
 <link name="aIR_FR">
   <collision>
-    <origin xyz="0 0 0" rpy="0 0 0"/>
+    <origin xyz="0 0 -0.00709" rpy="0 0 0"/>
     <geometry>
       <box size="0.01418 0.04839 0.013"/>
@@ -457,5 +459,5 @@
 <link name="aIR_FL">
   <collision>
-    <origin xyz="0 0 0" rpy="0 0 0"/>
+    <origin xyz="0 0 -0.00709" rpy="0 0 0"/>
     <geometry>
       <box size="0.01418 0.04839 0.013"/>
@@ -482,4 +484,86 @@
   <parent link="base_link"/>
   <child link="aIR_FL"/>
+</joint>
+<link name="sonic_FD">
+  <collision>
+    <origin xyz="0.00725 0 0" rpy="0 0 0"/>
+    <geometry>
+      <box size="0.0145 0.04572 0.02"/>
+    </geometry>
+  </collision>
+  <visual>
+    <origin xyz="0 0 0" rpy="0 0 0"/>
+    <geometry>
+      <mesh filename="package://devastator/devastator_description/meshes/sensors/ultrasonic.dae"/>
+    </geometry>
+  </visual>
+  <inertial>
+    <mass value="0.25" />
+    <origin xyz="0 0 0" rpy="0 0 0"/>
+    <box_inertia m="0.25" x="0.015" y="0.015" z="0.02" />
+    <inertia ixx="1.0e-6" ixy="0.0" ixz="0.0"
+    iyy="1.0e-6" iyz="0.0" izz="1.0e-6" />
+  </inertial>
+</link>
+<joint name="sonic_FD" type="fixed">
+  <axis xyz="0 0 1" />
+  <origin xyz="0.0992 0 0.03481" rpy="0 0 0"/>
+  <parent link="base_link"/>
+  <child link="sonic_FD"/>
+</joint>
+<link name="sonic_FF">
+  <collision>
+    <origin xyz="0.00725 0 0" rpy="0 0 0"/>
+    <geometry>
+      <box size="0.0145 0.04572 0.02"/>
+    </geometry>
+  </collision>
+  <visual>
+    <origin xyz="0 0 0" rpy="0 0 0"/>
+    <geometry>
+      <mesh filename="package://devastator/devastator_description/meshes/sensors/ultrasonic.dae"/>
+    </geometry>
+  </visual>
+  <inertial>
+    <mass value="0.25" />
+    <origin xyz="0 0 0" rpy="0 0 0"/>
+    <box_inertia m="0.25" x="0.015" y="0.015" z="0.02" />
+    <inertia ixx="1.0e-6" ixy="0.0" ixz="0.0"
+    iyy="1.0e-6" iyz="0.0" izz="1.0e-6" />
+  </inertial>
+</link>
+<joint name="sonic_FF" type="fixed">
+  <axis xyz="0 1 0" />
+  <origin xyz="0.07229 0.02739 0.10304" rpy="0 0.20944 0"/>
+  <parent link="base_link"/>
+  <child link="sonic_FF"/>
+</joint>
+<link name="dIR_FF">
+  <collision>
+    <axis xyz="0 1 0" />
+    <origin xyz="0.0085 0 0" rpy="0 -1.57 0"/>
+    <geometry>
+      <cylinder length="0.017" radius="0.0045"/>
+    </geometry>
+  </collision>
+  <visual>
+    <origin xyz="0 0 0" rpy="0 0 0"/>
+    <geometry>
+      <mesh filename="package://devastator/devastator_description/meshes/sensors/digital_ir.dae"/>
+    </geometry>
+  </visual>
+  <inertial>
+    <mass value="0.25" />
+    <origin xyz="0 0 0" rpy="0 0 0"/>
+    <box_inertia m="0.25" x="0.015" y="0.015" z="0.02" />
+    <inertia ixx="1.0e-6" ixy="0.0" ixz="0.0"
+    iyy="1.0e-6" iyz="0.0" izz="1.0e-6" />
+  </inertial>
+</link>
+<joint name="dIR_FF" type="fixed">
+  <axis xyz="0 1 0" />
+  <origin xyz="0.07229 0 0.10304" rpy="0 0.20944 0"/>
+  <parent link="base_link"/>
+  <child link="dIR_FF"/>
 </joint>
 <!--link name="hokuyo">
