Commit message: fixed full urdf, added gazebo plugin file, added empty world file for full model

File: devastator_description/urdf/devastator_full.gazebo.xacro (robot description, xacro)
@@ -17,4 +17,5 @@
     </plugin>
   </gazebo>
+<!--
   <gazebo reference="camera">
     <material>Gazebo/Red</material>
@@ -53,5 +54,5 @@
     <sensor type="ray" name="lds_lfcd_sensor">
       <pose>0 0 0 0 0 0</pose>
-      <!--visualize>$(arg laser_visual)</visualize-->
+      <visualize>$(arg laser_visual)</visualize>
       <visualize>false</visualize>
       <ray>
@@ -81,4 +82,4 @@
       </plugin>
     </sensor>
-  </gazebo>
+  </gazebo-->
 </robot>

File: devastator_description/urdf/devastator_full.urdf.xacro (robot description, xacro)
@@ -1,5 +1,5 @@
 <?xml version="1.0"?>
 <robot name="devastator" xmlns:xacro="http://www.ros.org/wiki/xacro">
-  <xacro:include filename="$(find devastator)/devastator_description/urdf/devastator_laser.gazebo.xacro" />
+  <xacro:include filename="$(find devastator)/devastator_description/urdf/devastator_full.gazebo.xacro" />
   <!--xacro:include filename="$(find mybot_description)/urdf/materials.xacro" /-->
   <xacro:include filename="$(find mybot_description)/urdf/macros.xacro" />

File: devastator_description/urdf/devastator_laser.urdf.xacro (robot description, xacro)
@@ -6,10 +6,4 @@
   <!--xacro:include filename="$(find mybot_description)/urdf/materials.xacro" /-->
   <xacro:include filename="$(find mybot_description)/urdf/macros.xacro" />
-<!--link name="base_footprint"/>
-  <joint name="base_joint" type="fixed">
-    <parent link="base_footprint"/>
-    <origin xyz="0.0 0.0 0.0" rpy="0 0 1.57"/>
-    <child link="base_link"/>
-  </joint-->
 <link name="base_link">
 	<visual>
@@ -376,30 +370,3 @@
     <child link="hokuyo"/>
   </joint>
-<!--link name="belt">
-	<visual>
-		<origin rpy="0 0 0" xyz="0 0 0"/>
-		<geometry>
-			<mesh filename="package://devastator/devastator_description/meshes/wheels/belt2.dae"/>
-		</geometry>
-	</visual>
-	<collision>
-		<origin xyz="0 0 0" rpy="0 0 0"/>
-		<geometry>
-			<cylinder length="0.018" radius="0.033"/>
-		</geometry>
-	</collision>
-	<inertial>
-	<mass value= "0.212"/>
-  <Inertia matrix>
-		<inertia ixx="1.0" ixy=" 0" ixz="0.0"
-		iyy="1.0 " iyz="0.0"
-		izz="1.0 " />
-	</inertial>
-</link>
-<joint name="belt" type="continuous">
-	<parent link="base_link"/>
-	<child link="belt"/>
-	<origin xyz="0 0 0" rpy="0 0 0"/>
-	<axis xyz="0 0 1"/>
-</joint -->
 </robot>
